Commit message: Controller working, reduced to 20Hz speed for now. Launchfile working, but messages and transforms need namespacing

File: basalt_sim/urdf/x500_ref.urdf (robot description, URDF)
Before this commit: robot x500, 1 links, 0 joints
Links:
- removed link x500
- added link x500_ref; visual mesh filename=package://basalt_sim/meshes/x500_decimated.dae
